Commit message: feat: update JAKA A5 vision servo integration workflow

File: src/jaka_a5/jaka_a5_description/urdf/gazebo.urdf.xacro (robot description, xacro)
@@ -1,13 +1,4 @@
 <?xml version="1.0"?>
 <robot xmlns:xacro="http://www.ros.org/wiki/xacro">
-  <!-- Gazebo ros2_control plugin -->
-  <xacro:macro name="gazebo_ros2_control" params="name">
-    <gazebo>
-      <plugin name="gazebo_ros2_control" filename="libgazebo_ros2_control.so">
-        <robotNamespace>/${name}</robotNamespace>
-        <robotParam>robot_description</robotParam>
-      </plugin>
-    </gazebo>
-  </xacro:macro>
   <!-- Apply gazebo materials to all links -->
   <gazebo reference="base_link">
@@ -33,4 +24,51 @@
   </gazebo>
   <!-- ros2_control plugin -->
-  <gazebo_ros2_control name="jaka_a5" />
+  <gazebo>
+    <plugin filename="gz_ros2_control-system" name="gz_ros2_control::GazeboSimROS2ControlPlugin">
+      <parameters>$(find jaka_a5_control)/config/ros2_controllers.yaml</parameters>
+      <ros>
+        <remapping>/controller_manager/robot_description:=/robot_description</remapping>
+      </ros>
+    </plugin>
+  </gazebo>
+  <!-- ============================================================
+       Eye-in-Hand Camera Sensor (Gazebo)
+       挂在 J6 末端，发布 /camera/image_raw + /camera/camera_info
+       ============================================================ -->
+  <gazebo reference="camera_link">
+    <sensor type="camera" name="camera_sensor">
+      <!-- 相机更新频率 Hz -->
+      <always_on>true</always_on>
+      <visualize>true</visualize>
+      <update_rate>15.0</update_rate>
+      <gz_frame_id>camera_optical_frame</gz_frame_id>
+      <!-- Place the sensor slightly in front of the housing to avoid self-occlusion. -->
+      <pose>0.028 0 0 0 0 0</pose>
+      <topic>/camera/image_raw</topic>
+      <camera>
+        <camera_info_topic>/camera/camera_info</camera_info_topic>
+        <!-- 水平视场角 ~60度 -->
+        <horizontal_fov>1.047</horizontal_fov>
+        <!-- 图像分辨率与格式 -->
+        <image>
+          <width>640</width>
+          <height>480</height>
+          <format>R8G8B8</format>
+        </image>
+        <!-- 裁剪平面（Near/Far Plane） -->
+        <clip>
+          <near>0.01</near>
+          <far>100</far>
+        </clip>
+        <!-- 畸变参数（默认无畸变） -->
+        <distortion>
+          <k1>0.0</k1>
+          <k2>0.0</k2>
+          <p1>0.0</p1>
+          <p2>0.0</p2>
+          <kc>0.0</kc>
+        </distortion>
+      </camera>
+    </sensor>
+  </gazebo>
 </robot>

File: src/jaka_a5/jaka_a5_description/urdf/jaka_a5.robot.xacro (robot description, xacro)
@@ -4,4 +4,5 @@
   <xacro:property name="PI" value="3.1415926535897931" />
   <xacro:property name="VELOCITY" value="3.665" />
+  <link name="world" />
   <!-- Base Link -->
   <link name="base_link">
@@ -219,11 +220,94 @@
     <limit lower="-6.28" upper="6.28" effort="1000" velocity="3.665" />
   </joint>
-  <!-- Eye-in-Hand Camera Mount (fake link for camera) -->
-  <link name="camera_link" />
+  <!-- Eye-in-Hand Camera Mount -->
+  <link name="camera_link">
+    <inertial>
+      <origin xyz="0 0 0" rpy="0 0 0" />
+      <mass value="0.08" />
+      <inertia ixx="1.8e-05" ixy="0.0" ixz="0.0" iyy="1.8e-05" iyz="0.0" izz="1.2e-05" />
+    </inertial>
+    <visual>
+      <origin xyz="0.0 0.0 0.0" rpy="0 0 0" />
+      <geometry>
+        <box size="0.045 0.03 0.03" />
+      </geometry>
+      <material name="camera_body">
+        <color rgba="0.1 0.1 0.1 1.0" />
+      </material>
+    </visual>
+    <visual>
+      <origin xyz="0.024 0.0 0.0" rpy="0 1.5708 0" />
+      <geometry>
+        <cylinder radius="0.009" length="0.01" />
+      </geometry>
+      <material name="camera_lens">
+        <color rgba="0.25 0.45 0.8 1.0" />
+      </material>
+    </visual>
+    <collision>
+      <origin xyz="0.0 0.0 0.0" rpy="0 0 0" />
+      <geometry>
+        <box size="0.045 0.03 0.03" />
+      </geometry>
+    </collision>
+  </link>
   <joint name="camera_joint" type="fixed">
-    <origin xyz="0 0 0.02" rpy="0 0 0" />
+    <origin xyz="0.055 0 0.045" rpy="0 0 0" />
     <parent link="J6" />
     <child link="camera_link" />
   </joint>
+  <link name="camera_optical_frame" />
+  <joint name="camera_optical_joint" type="fixed">
+    <origin xyz="0 0 0" rpy="-1.57079632679 0 -1.57079632679" />
+    <parent link="camera_link" />
+    <child link="camera_optical_frame" />
+  </joint>
+  <ros2_control name="GazeboSimSystem" type="system">
+    <hardware>
+      <plugin>gz_ros2_control/GazeboSimSystem</plugin>
+    </hardware>
+    <joint name="joint_1">
+      <command_interface name="position" />
+      <state_interface name="position">
+        <param name="initial_value">0.20943951023931953</param>
+      </state_interface>
+      <state_interface name="velocity" />
+    </joint>
+    <joint name="joint_2">
+      <command_interface name="position" />
+      <state_interface name="position">
+        <param name="initial_value">1.9198621771937625</param>
+      </state_interface>
+      <state_interface name="velocity" />
+    </joint>
+    <joint name="joint_3">
+      <command_interface name="position" />
+      <state_interface name="position">
+        <param name="initial_value">-2.181661564992912</param>
+      </state_interface>
+      <state_interface name="velocity" />
+    </joint>
+    <joint name="joint_4">
+      <command_interface name="position" />
+      <state_interface name="position">
+        <param name="initial_value">0.3141592653589793</param>
+      </state_interface>
+      <state_interface name="velocity" />
+    </joint>
+    <joint name="joint_5">
+      <command_interface name="position" />
+      <state_interface name="position">
+        <param name="initial_value">0.22689280275926285</param>
+      </state_interface>
+      <state_interface name="velocity" />
+    </joint>
+    <joint name="joint_6">
+      <command_interface name="position" />
+      <state_interface name="position">
+        <param name="initial_value">0.0</param>
+      </state_interface>
+      <state_interface name="velocity" />
+    </joint>
+  </ros2_control>
   <!-- ROS2 control transmission - repeat for all 6 joints -->
   <transmission name="trans_joint_1">

File: src/jaka_a5/jaka_a5_description/urdf/jaka_a5.urdf.xacro (robot description, xacro)
@@ -1,4 +1,3 @@
 <?xml version="1.0"?>
-<?xml-model href="http://www.ros.org/wiki/xacro" ?>
 <robot xmlns:xacro="http://www.ros.org/wiki/xacro"
        name="jaka_a5">
